File: wr02sd/wr02sd.sch (KiCad schematic (older format))
At the start: 9 parts

Commit message: PCB Artworking is progressing.
Parts:
- removed CON?: Micro_SD_Card, symbol Micro_SD_Card
- added C4, C8: 100u, Capacitors_Tantalum_SMD:TantalC_SizeS_EIA-3216, symbol CP_Small
- added C5: 0.47u, Capacitors_SMD:C_1206, symbol C_Small
- added C6: 10u, Capacitors_SMD:C_1206, symbol CP_Small
- added C7: 47u, Capacitors_SMD:C_1210, symbol CP_Small
- added C9: 470, Capacitors_SMD:C_0805, symbol C_Small
- added CON1: SD_Card, wroom02:MICROSD, symbol SD_Card
- added D1: IN4007/M7(DO-214AC), Diodes_SMD:DO-214AB, symbol D_Schottky_Small
- added P1, P3: THT_Male_P_1x15, Pin_Headers:Pin_Header_Straight_1x15, symbol CONN_01X15
- added P4: POWER_5V, Connectors_JST:JST_PH_B2B-PH-K_02x2.00mm_Straight, symbol CONN_01X02
- added R1: 220K(1%), Resistors_SMD:R_0402, symbol R_Small
- added R2: 100K(1%), Resistors_SMD:R_0402, symbol R_Small
- added R4, R5, R6, R7, R8, R9: 10K, Resistors_SMD:R_0201, symbol R_Small
- added SW1: Flash, Buttons_Switches_SMD:SW_SPST_B3U-1000P, symbol SW_PUSH_SMALL_H
- added SW2: Reset, Buttons_Switches_SMD:SW_SPST_B3U-1000P, symbol SW_PUSH_SMALL_H
- added U2: LM3940IMP-3.3, TO_SOT_Packages_SMD:SOT-223, symbol LM3940IMP-3.3
- C1, C2: renamed from C?; footprint (none) -> Capacitors_SMD:C_0201
- C3: renamed from C?; footprint (none) -> Capacitors_SMD:C_1206
- P2: renamed from P?; footprint (none) -> Connect:USB_Micro-B
- R3: renamed from R?; footprint (none) -> Resistors_SMD:R_0201
- U1: renamed from U?; footprint (none) -> Housings_SOIC:SOIC-16_3.9x9.9mm_Pitch1.27mm
- U3: renamed from U?; footprint (none) -> wroom02:ESP-13-WROOM-02
- Y1: renamed from Y?; footprint (none) -> wroom02:smd_xtal
Connections:
- net labels added: +5V, ADC, EN, GPIO0, GPIO12(MISO), GPIO13(MOSI), GPIO14(CK), GPIO15(CD), GPIO16, GPIO2, GPIO4, GPIO5, USB_D+, USB_D-, VDD, nRST
- net labels removed: SPI_CD, SPI_CK, SPI_MISO, SPI_MOSI
- wire segments 45 -> 136
- no-connect marks 9 -> 16
Other:
- note added: "Matter NEEDED Attention\nOn every boot/reset/wakeup,\nGPIO15 MUST keep LOW, GPIO2 MUST keep HIGH,\nGPIO0 HIGH -> Run mode, LOW -> Flash mode.\nWhen you need to use the sleep mode, GPIO16 and RST shud be connected,\nand GPIO16 will output LOW to reset the system at the time of wakeup."
- moved on the sheet: C1, C2, C3, P2, R3, U1, U3, Y1

Commit message: PCB Artworking is progressing..
Parts:
- removed CON1: SD_Card, wroom02:MICROSD, symbol SD_Card
- added CON1: Micro_SD_Card, wroom02:MICROSD, symbol Micro_SD_Card
Connections:
- wire segments 136 -> 132
- no-connect marks 16 -> 14
Other:
- moved on the sheet: C3
Changed lines of the file:
@@
 	1    0    0    -1
 $EndComp
-NoConn ~ 3050 4800
-Text Label 3450 4500 0    60   ~ 0
+NoConn ~ 3050 4700
+Text Label 3450 4400 0    60   ~ 0
 GPIO14(CK)
-Text Label 3350 4700 0    60   ~ 0
+Text Label 3350 4600 0    60   ~ 0
 GPIO12(MISO)
 Text Label 3350 4200 0    60   ~ 0
@@
 L CP_Small C3
 U 1 1 57BD60BD
-P 4250 4500
-F 0 "C3" H 4350 4550 50  0000 L CNN
-F 1 "10u" H 4350 4450 50  0000 L CNN
-F 2 "Capacitors_SMD:C_1206" H 4250 4500 50  0001 C CNN
-F 3 "" H 4250 4500 50  0000 C CNN
-	1    4250 4500
+P 4250 4400
+F 0 "C3" H 4350 4450 50  0000 L CNN
+F 1 "10u" H 4350 4350 50  0000 L CNN
+F 2 "Capacitors_SMD:C_1206" H 4250 4400 50  0001 C CNN
+F 3 "" H 4250 4400 50  0000 C CNN
+	1    4250 4400
 	1    0    0    -1
 $EndComp
@@
 L GND #PWR06
 U 1 1 57BD62C3
-P 4250 4750
-F 0 "#PWR06" H 4250 4500 50  0001 C CNN
-F 1 "GND" H 4250 4600 50  0000 C CNN
-F 2 "" H 4250 4750 50  0000 C CNN
-F 3 "" H 4250 4750 50  0000 C CNN
-	1    4250 4750
+P 4250 4650
+F 0 "#PWR06" H 4250 4400 50  0001 C CNN
+F 1 "GND" H 4250 4500 50  0000 C CNN
+F 2 "" H 4250 4650 50  0000 C CNN
+F 3 "" H 4250 4650 50  0000 C CNN
+	1    4250 4650
 	1    0    0    -1
 $EndComp
@@
 L VCC #PWR07
 U 1 1 57BD62EE
-P 4250 4200
-F 0 "#PWR07" H 4250 4050 50  0001 C CNN
-F 1 "VCC" H 4250 4350 50  0000 C CNN
-F 2 "" H 4250 4200 50  0000 C CNN
-F 3 "" H 4250 4200 50  0000 C CNN
-	1    4250 4200
+P 4250 4100
+F 0 "#PWR07" H 4250 3950 50  0001 C CNN
+F 1 "VCC" H 4250 4250 50  0000 C CNN
+F 2 "" H 4250 4100 50  0000 C CNN
+F 3 "" H 4250 4100 50  0000 C CNN
+	1    4250 4100
 	1    0    0    -1
 $EndComp
@@
 	3050 3300 2550 3300
 Wire Wire Line
-	3050 4400 4250 4400
-Wire Wire Line
-	4250 4400 4250 4200
-Wire Wire Line
-	3050 4600 4250 4600
-Wire Wire Line
-	4250 4600 4250 4750
+	3050 4300 4250 4300
+Wire Wire Line
+	4250 4300 4250 4100
+Wire Wire Line
+	3050 4500 4250 4500
+Wire Wire Line
+	4250 4500 4250 4650
 Wire Wire Line
 	7350 2200 5500 2200
@@
 	5500 2100 7350 2100
 Wire Wire Line
-	3950 4700 3050 4700
+	3950 4600 3050 4600
 Wire Wire Line
 	5500 2300 7350 2300
@@
 	7350 2000 5500 2000
 Wire Wire Line
-	3950 4500 3050 4500
-Connection ~ 4250 4400
-Connection ~ 4250 4600
+	3950 4400 3050 4400
+Connection ~ 4250 4300
+Connection ~ 4250 4500
 Wire Wire Line
 	2550 3300 2550 3200
@@
 Connection ~ 4700 5500
 $Comp
-L SD_Card CON1
-U 1 1 57BE9D62
-P 2150 4400
-F 0 "CON1" H 1500 4950 50  0000 C CNN
-F 1 "SD_Card" H 2750 3850 50  0000 C CNN
-F 2 "wroom02:MICROSD" H 2350 4750 50  0000 C CNN
-F 3 "" H 2150 4400 50  0000 C CNN
-	1    2150 4400
-	-1   0    0    -1
-$EndComp
-NoConn ~ 3050 4000
-Wire Wire Line
-	3050 4300 3150 4300
-Wire Wire Line
-	3150 4300 3150 4600
-Connection ~ 3150 4600
-$Comp
 L GND #PWR035
 U 1 1 57BEA6E2
-P 1200 4850
-F 0 "#PWR035" H 1200 4600 50  0001 C CNN
-F 1 "GND" H 1200 4700 50  0000 C CNN
-F 2 "" H 1200 4850 50  0000 C CNN
-F 3 "" H 1200 4850 50  0000 C CNN
-	1    1200 4850
-	1    0    0    -1
-$EndComp
-Wire Wire Line
-	1200 4500 1200 4850
-Wire Wire Line
-	1250 4500 1200 4500
-Wire Wire Line
-	1250 4600 1200 4600
-Connection ~ 1200 4600
-NoConn ~ 1250 4200
-NoConn ~ 1250 4300
+P 1350 5050
+F 0 "#PWR035" H 1350 4800 50  0001 C CNN
+F 1 "GND" H 1350 4900 50  0000 C CNN
+F 2 "" H 1350 5050 50  0000 C CNN
+F 3 "" H 1350 5050 50  0000 C CNN
+	1    1350 5050
+	1    0    0    -1
+$EndComp
+NoConn ~ 3050 4000
+$Comp
+L Micro_SD_Card CON1
+U 1 1 57BF871D
+P 2150 4300
+F 0 "CON1" H 1500 4900 50  0000 C CNN
+F 1 "Micro_SD_Card" H 2800 4900 50  0000 R CNN
+F 2 "wroom02:MICROSD" H 3300 4600 50  0001 C CNN
+F 3 "" H 2150 4300 50  0000 C CNN
+	1    2150 4300
+	-1   0    0    -1
+$EndComp
+Wire Wire Line
+	1350 4900 1350 5050
 $EndSCHEMATC

Commit message: PCB Artworking the first is done.
Parts:
- P2: footprint Connect:USB_Micro-B -> wroom02:uUSB_B_Receptacle
Connections:
- wire segments 132 -> 130
- no-connect marks 14 -> 15
Other:
- moved on the sheet: R9
Changed lines of the file:
@@
 F 0 "P2" H 1850 2150 50  0000 C CNN
 F 1 "USB_A" H 1600 2550 50  0000 C CNN
-F 2 "Connect:USB_Micro-B" V 1600 2250 50  0001 C CNN
+F 2 "wroom02:uUSB_B_Receptacle" V 1600 2250 50  0001 C CNN
 F 3 "" V 1600 2250 50  0000 C CNN
 	1    1650 2350
@@
 L GND #PWR01
 U 1 1 57BD53F5
-P 1950 2750
-F 0 "#PWR01" H 1950 2500 50  0001 C CNN
-F 1 "GND" H 1950 2600 50  0000 C CNN
-F 2 "" H 1950 2750 50  0000 C CNN
-F 3 "" H 1950 2750 50  0000 C CNN
-	1    1950 2750
+P 1550 2750
+F 0 "#PWR01" H 1550 2500 50  0001 C CNN
+F 1 "GND" H 1550 2600 50  0000 C CNN
+F 2 "" H 1550 2750 50  0000 C CNN
+F 3 "" H 1550 2750 50  0000 C CNN
+	1    1550 2750
 	1    0    0    -1
 $EndComp
@@
 L R_Small R9
 U 1 1 57BE3F5D
-P 7750 3750
-F 0 "R9" V 7650 3650 50  0000 L CNN
-F 1 "10K" V 7850 3700 50  0000 L CNN
-F 2 "Resistors_SMD:R_0201" H 7750 3750 50  0001 C CNN
-F 3 "" H 7750 3750 50  0000 C CNN
-	1    7750 3750
-	0    1    1    0
+P 9550 1750
+F 0 "R9" V 9450 1650 50  0000 L CNN
+F 1 "10K" V 9650 1700 50  0000 L CNN
+F 2 "Resistors_SMD:R_0201" H 9550 1750 50  0001 C CNN
+F 3 "" H 9550 1750 50  0000 C CNN
+	1    9550 1750
+	1    0    0    -1
 $EndComp
 $Comp
@@
 	1950 1850 1950 2150
 Wire Wire Line
-	1950 2450 1950 2750
-Wire Wire Line
 	3500 1950 2850 1950
 Wire Wire Line
@@
 	2550 2250 2300 2350
 Wire Wire Line
-	1550 2650 1550 2700
-Wire Wire Line
-	1550 2700 1950 2700
-Connection ~ 1950 2700
+	1550 2650 1550 2750
 Wire Wire Line
 	4850 1150 4850 1850
@@
 	7100 3350 7100 3450
 Wire Wire Line
-	9550 2100 9550 3750
-Wire Wire Line
-	9550 3750 7850 3750
+	9550 1850 9550 3750
 Connection ~ 9550 2100
 Wire Wire Line
 	7100 3650 7100 3750
 Wire Wire Line
-	7550 3750 7650 3750
+	9550 3750 7550 3750
 $Comp
 L CONN_01X15 P1
@@
 Text Notes 6950 4450 0    50   ~ 0
 Matter NEEDED Attention\nOn every boot/reset/wakeup,\nGPIO15 MUST keep LOW, GPIO2 MUST keep HIGH,\nGPIO0 HIGH -> Run mode, LOW -> Flash mode.\nWhen you need to use the sleep mode, GPIO16 and RST shud be connected,\nand GPIO16 will output LOW to reset the system at the time of wakeup.
-Text Label 8000 3750 0    60   ~ 0
+Text Label 7650 3750 0    60   ~ 0
 nRST
 Text Label 6950 3050 1    60   ~ 0
@@
 Wire Wire Line
 	1350 4900 1350 5050
+$Comp
+L VCC #PWR036
+U 1 1 57C5171C
+P 9550 1600
+F 0 "#PWR036" H 9550 1450 50  0001 C CNN
+F 1 "VCC" H 9550 1750 50  0000 C CNN
+F 2 "" H 9550 1600 50  0000 C CNN
+F 3 "" H 9550 1600 50  0000 C CNN
+	1    9550 1600
+	1    0    0    -1
+$EndComp
+Wire Wire Line
+	9550 1600 9550 1650
+NoConn ~ 1950 2450
 $EndSCHEMATC

Commit message: 更新
Parts:
- removed C9: 470, Capacitors_SMD:C_0805, symbol C_Small
- added C9: 10u, Capacitors_SMD:C_0603, symbol C
Connections:
- wire segments 130 -> 132
Other:
- note added: "(10u)"
- note added: "(1u)"
- note added: "(22u)"
- note added: "(INT)"
- note added: "(SCL)"
- note added: "(SDA)"
Changed lines of the file:
@@
 LIBS:memory
 LIBS:wr02sd
+LIBS:philips
 LIBS:wr02sd-cache
 EELAYER 25 0
@@
 $Descr A4 11693 8268
 encoding utf-8
-Sheet 1 1
-Title "WROOM02-SDCard break out board"
-Date "2016-08-24"
-Rev "01A"
+Sheet 1 2
+Title "gpio-keypad"
+Date "2016-10-05"
+Rev "a"
 Comp "Mazzacraft"
 Comment1 ""
@@
 $EndComp
 $Comp
-L C_Small C9
-U 1 1 57BE4A77
-P 7450 3750
-F 0 "C9" V 7350 3750 50  0000 L CNN
-F 1 "470" V 7550 3700 50  0000 L CNN
-F 2 "Capacitors_SMD:C_0805" H 7450 3750 50  0001 C CNN
-F 3 "" H 7450 3750 50  0000 C CNN
-	1    7450 3750
-	0    -1   1    0
-$EndComp
-$Comp
 L GND #PWR011
 U 1 1 57BE4CB2
@@
 	7100 3350 7100 3450
 Wire Wire Line
-	9550 1850 9550 3750
+	9550 1850 9550 2100
+Wire Wire Line
+	9550 2100 9540 3750
 Connection ~ 9550 2100
 Wire Wire Line
 	7100 3650 7100 3750
 Wire Wire Line
-	9550 3750 7550 3750
+	9540 3750 7650 3750
 $Comp
 L CONN_01X15 P1
@@
 	3500 6200 4150 6200
 Wire Wire Line
-	3500 6300 4300 6300
-Wire Wire Line
-	4700 6400 3500 6400
-Wire Wire Line
-	3500 6500 4150 6500
+	3500 6300 4250 6300
+Wire Wire Line
+	3500 6400 4850 6400
+Wire Wire Line
+	3500 6500 4850 6500
 Wire Wire Line
 	3500 6600 4150 6600
 Wire Wire Line
-	3500 6700 4150 6700
-Wire Wire Line
-	3500 6800 4150 6800
+	3500 6700 4850 6700
+Wire Wire Line
+	3500 6800 4850 6800
 Wire Wire Line
 	3500 6900 4150 6900
@@
 GPIO16
 Wire Wire Line
-	3500 5500 4700 5500
-Wire Wire Line
-	3500 5600 4300 5600
-Text Label 4650 6400 2    60   ~ 0
+	3500 5500 4650 5500
+Wire Wire Line
+	3500 5600 4250 5600
+Text Label 4500 5500 2    60   ~ 0
 VCC
-Text Label 4650 5500 2    60   ~ 0
-VCC
-Wire Wire Line
-	4300 5600 4300 6500
-Connection ~ 4300 6300
-$Comp
-L GND #PWR020
-U 1 1 57BEC9BC
-P 4300 6500
-F 0 "#PWR020" H 4300 6250 50  0001 C CNN
-F 1 "GND" H 4300 6350 50  0000 C CNN
-F 2 "" H 4300 6500 50  0000 C CNN
-F 3 "" H 4300 6500 50  0000 C CNN
-	1    4300 6500
-	-1   0    0    -1
-$EndComp
+Wire Wire Line
+	4250 5600 4250 7150
+Connection ~ 4250 6300
 Text Label 2550 2250 0    60   ~ 0
 USB_D+
@@
 Connection ~ 7900 5400
 $Comp
-L GND #PWR021
+L GND #PWR020
 U 1 1 57BEE657
 P 7300 5900
-F 0 "#PWR021" H 7300 5650 50  0001 C CNN
+F 0 "#PWR020" H 7300 5650 50  0001 C CNN
 F 1 "GND" H 7300 5750 50  0000 C CNN
 F 2 "" H 7300 5900 50  0000 C CNN
@@
 $EndComp
 $Comp
-L VCC #PWR022
+L VCC #PWR021
 U 1 1 57BEED7C
 P 7900 5350
-F 0 "#PWR022" H 7900 5200 50  0001 C CNN
+F 0 "#PWR021" H 7900 5200 50  0001 C CNN
 F 1 "VCC" H 7900 5500 50  0000 C CNN
 F 2 "" H 7900 5350 50  0000 C CNN
@@
 $EndComp
 $Comp
-L PWR_FLAG #FLG023
+L PWR_FLAG #FLG022
 U 1 1 57BEFDC3
 P 9300 5500
-F 0 "#FLG023" H 9300 5595 50  0001 C CNN
+F 0 "#FLG022" H 9300 5595 50  0001 C CNN
 F 1 "PWR_FLAG" H 9300 5680 50  0000 C CNN
 F 2 "" H 9300 5500 50  0000 C CNN
@@
 $EndComp
 $Comp
-L PWR_FLAG #FLG024
+L PWR_FLAG #FLG023
 U 1 1 57BEFE22
 P 8850 5500
-F 0 "#FLG024" H 8850 5595 50  0001 C CNN
+F 0 "#FLG023" H 8850 5595 50  0001 C CNN
 F 1 "PWR_FLAG" H 8850 5680 50  0000 C CNN
 F 2 "" H 8850 5500 50  0000 C CNN
@@
 $EndComp
 $Comp
-L GND #PWR025
+L GND #PWR024
 U 1 1 57BEFE81
 P 8850 5650
-F 0 "#PWR025" H 8850 5400 50  0001 C CNN
+F 0 "#PWR024" H 8850 5400 50  0001 C CNN
 F 1 "GND" H 8850 5500 50  0000 C CNN
 F 2 "" H 8850 5650 50  0000 C CNN
@@
 $EndComp
 $Comp
-L VDD #PWR026
+L VDD #PWR025
 U 1 1 57BEFF3F
 P 9300 5650
-F 0 "#PWR026" H 9300 5500 50  0001 C CNN
+F 0 "#PWR025" H 9300 5500 50  0001 C CNN
 F 1 "VDD" H 9300 5800 50  0000 C CNN
 F 2 "" H 9300 5650 50  0000 C CNN
@@
 	8850 5500 8850 5650
 $Comp
-L GND #PWR027
+L GND #PWR026
 U 1 1 57BF0A08
 P 8350 3100
-F 0 "#PWR027" H 8350 2850 50  0001 C CNN
+F 0 "#PWR026" H 8350 2850 50  0001 C CNN
 F 1 "GND" H 8350 2950 50  0000 C CNN
 F 2 "" H 8350 3100 50  0000 C CNN
@@
 	8350 3000 8350 3100
 $Comp
-L PWR_FLAG #FLG028
+L PWR_FLAG #FLG027
 U 1 1 57BF0D71
 P 9750 5500
-F 0 "#FLG028" H 9750 5595 50  0001 C CNN
+F 0 "#FLG027" H 9750 5595 50  0001 C CNN
 F 1 "PWR_FLAG" H 9750 5680 50  0000 C CNN
 F 2 "" H 9750 5500 50  0000 C CNN
@@
 $EndComp
 $Comp
-L +5V #PWR029
+L +5V #PWR028
 U 1 1 57BF0DD0
 P 9750 5650
-F 0 "#PWR029" H 9750 5500 50  0001 C CNN
+F 0 "#PWR028" H 9750 5500 50  0001 C CNN
 F 1 "+5V" H 9750 5790 50  0000 C CNN
 F 2 "" H 9750 5650 50  0000 C CNN
@@
 $EndComp
 $Comp
-L +5V #PWR030
+L +5V #PWR029
 U 1 1 57BF1676
 P 5800 5200
-F 0 "#PWR030" H 5800 5050 50  0001 C CNN
+F 0 "#PWR029" H 5800 5050 50  0001 C CNN
 F 1 "+5V" H 5800 5340 50  0000 C CNN
 F 2 "" H 5800 5200 50  0000 C CNN
@@
 Connection ~ 6700 5800
 $Comp
-L VDD #PWR031
+L VDD #PWR030
 U 1 1 57BF27E4
 P 6200 5650
-F 0 "#PWR031" H 6200 5500 50  0001 C CNN
+F 0 "#PWR030" H 6200 5500 50  0001 C CNN
 F 1 "VDD" H 6200 5800 50  0000 C CNN
 F 2 "" H 6200 5650 50  0000 C CNN
@@
 	6200 5700 6200 5650
 $Comp
-L VDD #PWR032
+L VDD #PWR031
 U 1 1 57BF2AD0
 P 2800 5450
-F 0 "#PWR032" H 2800 5300 50  0001 C CNN
+F 0 "#PWR031" H 2800 5300 50  0001 C CNN
 F 1 "VDD" H 2800 5600 50  0000 C CNN
 F 2 "" H 2800 5450 50  0000 C CNN
@@
 	2800 5450 2800 5500
 $Comp
-L VCC #PWR033
+L VCC #PWR032
 U 1 1 57BF2D4A
 P 2800 5850
-F 0 "#PWR033" H 2800 5700 50  0001 C CNN
+F 0 "#PWR032" H 2800 5700 50  0001 C CNN
 F 1 "VCC" H 2800 6000 50  0000 C CNN
 F 2 "" H 2800 5850 50  0000 C CNN
@@
 	2800 5900 2800 5850
 $Comp
-L VCC #PWR034
+L VCC #PWR033
 U 1 1 57BF2F8A
-P 4700 5450
-F 0 "#PWR034" H 4700 5300 50  0001 C CNN
-F 1 "VCC" H 4700 5600 50  0000 C CNN
-F 2 "" H 4700 5450 50  0000 C CNN
-F 3 "" H 4700 5450 50  0000 C CNN
-	1    4700 5450
-	1    0    0    -1
-$EndComp
-Wire Wire Line
-	4700 5450 4700 6400
-Connection ~ 4700 5500
-$Comp
-L GND #PWR035
+P 4650 5500
+F 0 "#PWR033" H 4650 5350 50  0001 C CNN
+F 1 "VCC" H 4650 5650 50  0000 C CNN
+F 2 "" H 4650 5500 50  0000 C CNN
+F 3 "" H 4650 5500 50  0000 C CNN
+	1    4650 5500
+	1    0    0    -1
+$EndComp
+Wire Wire Line
+	4650 5500 4650 6400
+Connection ~ 4650 5500
+$Comp
+L GND #PWR034
 U 1 1 57BEA6E2
 P 1350 5050
-F 0 "#PWR035" H 1350 4800 50  0001 C CNN
+F 0 "#PWR034" H 1350 4800 50  0001 C CNN
 F 1 "GND" H 1350 4900 50  0000 C CNN
 F 2 "" H 1350 5050 50  0000 C CNN
@@
 	1350 4900 1350 5050
 $Comp
-L VCC #PWR036
+L VCC #PWR035
 U 1 1 57C5171C
 P 9550 1600
-F 0 "#PWR036" H 9550 1450 50  0001 C CNN
+F 0 "#PWR035" H 9550 1450 50  0001 C CNN
 F 1 "VCC" H 9550 1750 50  0000 C CNN
 F 2 "" H 9550 1600 50  0000 C CNN
@@
 	9550 1600 9550 1650
 NoConn ~ 1950 2450
+Text Notes 6800 5750 0    60   ~ 0
+(1u)
+Text Notes 7950 5800 0    60   ~ 0
+(22u)
+Text Notes 6750 1400 0    60   ~ 0
+(10u)
+$Sheet
+S 4850 6350 550  700
+U 57F44A49
+F0 "keypad" 60
+F1 "keypad.sch" 60
+F2 "VCC" B L 4850 6400 60
+F3 "GND" B L 4850 7000 60
+F4 "GPIO4" B L 4850 6700 60
+F5 "GPIO2" B L 4850 6500 60
+F6 "GPIO5" B L 4850 6800 60
+$EndSheet
+Text Notes 3600 6500 0    60   Italic 0
+(SDA)
+Text Notes 3600 6700 0    60   Italic 0
+(SCL)
+Text Notes 3600 6800 0    60   Italic 0
+(INT)
+$Comp
+L GND #PWR036
+U 1 1 57BEC9BC
+P 4250 7150
+F 0 "#PWR036" H 4250 6900 50  0001 C CNN
+F 1 "GND" H 4250 7000 50  0000 C CNN
+F 2 "" H 4250 7150 50  0000 C CNN
+F 3 "" H 4250 7150 50  0000 C CNN
+	1    4250 7150
+	-1   0    0    -1
+$EndComp
+Wire Wire Line
+	4850 7000 4250 7000
+Connection ~ 4250 7000
+Connection ~ 4650 6400
+$Comp
+L C C9
+U 1 1 5818494F
+P 7500 3750
+F 0 "C9" V 7345 3705 50  0000 L CNN
+F 1 "10u" V 7625 3665 50  0000 L CNN
+F 2 "Capacitors_SMD:C_0603" H 7538 3600 50  0001 C CNN
+F 3 "" H 7500 3750 50  0000 C CNN
+	1    7500 3750
+	0    1    1    0
+$EndComp
 $EndSCHEMATC
